Commit message: Fixing launch issues and adding no leg model. Need to make prismatic joint raise and lower the base.

File: urdf/human-no-legs.xacro (robot description, xacro)
@@ -18,4 +18,5 @@
     <xacro:property name="tight_length" value="${size_unit*1.5}" />
     <xacro:property name="tibia_length" value="${size_unit*2}" />
+    <xacro:property name="leg_length" value="${size_unit*2 + size_unit*1.5}" />
     <xacro:property name="limb_radius" value="0.03" />
     <!-- Materials -->
@@ -30,16 +31,29 @@
     </material>
     <!--***********-->
+    <!-- <link name="world" /> -->
     <link name="body_${id}">
     </link>
+    <!-- <joint name="base_joint" type="fixed">
+        <parent link="world" />
+        <child link="body_${id}" />
+    </joint> -->
     <link name="waist_${id}">
     </link>
+    <link name="waist_intermediate_${id}">
+    </link>
     <link name="torso_${id}">
         <visual>
             <geometry>
-                <cylinder length="${3 * torso_height / 4}" radius="${limb_radius}"/>
+                <cylinder length="${torso_height}" radius="${limb_radius}"/>
             </geometry>
             <material name="yellow-skin" />
-            <origin rpy="0 0 0" xyz="0 0 -${3 * torso_height / 8}" />
-        </visual>
+            <origin rpy="0 0 0" xyz="0 0 -${torso_height / 2}" />
+        </visual>
+        <collision>
+            <geometry>
+                <cylinder length="${torso_height}" radius="${limb_radius}"/>
+            </geometry>
+            <origin rpy="0 0 0" xyz="0 0 -${torso_height / 2}" />
+        </collision>
         <visual>
             <geometry>
@@ -49,18 +63,10 @@
             <origin rpy="${pi / 2} 0 0" xyz="0 0 0" />
         </visual>
-        <visual>
-            <geometry>
-                <cylinder length="${waist_length/1.41}" radius="${limb_radius}"/>
-            </geometry>
-            <material name="yellow-skin" />
-            <origin rpy="${-pi / 4} 0 0" xyz="0 -${waist_length / 4} -${7 * torso_height / 8}" />
-        </visual>
-        <visual>
-            <geometry>
-                <cylinder length="${waist_length/1.41}" radius="${limb_radius}"/>
-            </geometry>
-            <material name="yellow-skin" />
-            <origin rpy="${pi / 4} 0 0" xyz="0 ${waist_length / 4} -${7 * torso_height / 8}" />
-        </visual>
+        <collision>
+            <geometry>
+                <cylinder length="${2 * neck_shoulder_length}" radius="${limb_radius}"/>
+            </geometry>
+            <origin rpy="${pi / 2} 0 0" xyz="0 0 0" />
+        </collision>
         <visual>
             <geometry>
@@ -70,4 +76,10 @@
             <origin rpy="0 0 0" xyz="0 0 -${3 * torso_height / 4}" />
         </visual>
+        <collision>
+            <geometry>
+                <sphere radius="${limb_radius}"/>
+            </geometry>
+            <origin rpy="0 0 0" xyz="0 0 -${3 * torso_height / 4}" />
+        </collision>
     </link>
     <joint name="torso_${id}" type="fixed">
@@ -76,8 +88,15 @@
         <origin rpy="0 0 0" xyz="0 0 ${torso_height}" />
     </joint>
+    <joint name="waist_${id}_z" type="revolute">
+        <axis xyz="0 0 1" />
+        <limit effort="1000" lower="-.4" upper="0.4" velocity="0.5" />
+        <parent link="body_${id}"/>
+        <child link="waist_intermediate_${id}"/>
+        <origin rpy="0 0 0" xyz="0 0 0" />
+    </joint>
     <joint name="waist_${id}" type="revolute">
         <axis xyz="0 1 0" />
         <limit effort="1000" lower="-.2" upper="1." velocity="0.5" />
-        <parent link="body_${id}"/>
+        <parent link="waist_intermediate_${id}"/>
         <child link="waist_${id}"/>
         <origin rpy="0 0 0" xyz="0 0 0" />
@@ -97,4 +116,10 @@
             <origin rpy="0 0 0" xyz="${-head_radius/2} 0 0" />
         </visual>
+        <collision>
+            <geometry>
+                <sphere radius="${head_radius}"/>
+            </geometry>
+            <origin rpy="0 0 0" xyz="${-head_radius/2} 0 0" />
+        </collision>
         <!-- eyes -->
         <visual>
@@ -148,4 +173,10 @@
                 <origin rpy="0 0 0" xyz="0 0 -${length/2}" />
             </visual>
+            <collision>
+                <geometry>
+                    <cylinder length="${length}" radius="${limb_radius}"/>
+                </geometry>
+                <origin rpy="0 0 0" xyz="0 0 -${length/2}" />
+            </collision>
             <visual>
                 <geometry>
@@ -155,4 +186,10 @@
                 <origin rpy="0 0 0" xyz="0 0 -${length}" />
             </visual>
+            <collision>
+                <geometry>
+                    <sphere radius="${limb_radius}"/>
+                </geometry>
+                <origin rpy="0 0 0" xyz="0 0 -${length}" />
+            </collision>
         </link>
         <joint name="${joint_name}" type="revolute">
@@ -167,10 +204,16 @@
         <link name="${suffix}_y_shoulder_${id}">
             <visual>
-            <geometry>
-                <sphere radius="${limb_radius}"/>
-            </geometry>
-            <material name="yellow-skin-dark" />
-            <origin rpy="0 0 0" xyz="0 0 0" />
-        </visual>
+                <geometry>
+                    <sphere radius="${limb_radius}"/>
+                </geometry>
+                <material name="yellow-skin-dark" />
+                <origin rpy="0 0 0" xyz="0 0 0" />
+            </visual>
+            <collision>
+                <geometry>
+                    <sphere radius="${limb_radius}"/>
+                </geometry>
+                <origin rpy="0 0 0" xyz="0 0 0" />
+            </collision>
         </link>
         <joint name="${suffix}_y_shoulder_${id}" type="revolute">
@@ -220,59 +263,61 @@
     <xacro:arm suffix="l" reflect="1" parent="torso_${id}" />
     <xacro:arm suffix="r" reflect="-1" parent="torso_${id}" />
-    <xacro:macro name="leg" params="suffix parent reflect">
-        <link name="${suffix}_y_hip_${id}">
-            <visual>
-            <geometry>
-                <sphere radius="${limb_radius}"/>
-            </geometry>
-            <material name="yellow-skin-dark" />
+    <xacro:macro name="single_leg" params="suffix parent">
+        <link name="${suffix}_leg_connector_${id}">
+            <visual>
+                <geometry>
+                    <sphere radius="${limb_radius}" />
+                </geometry>
+                <material name="yellow-skin-dark" />
+                <origin rpy="0 0 0" xyz="0 0 0" />
+            </visual>
+            <collision>
+                <geometry>
+                    <sphere radius="${limb_radius}" />
+                </geometry>
+                <origin rpy="0 0 0" xyz="0 0 0" />
+            </collision>
+        </link>
+        <joint name="${suffix}_leg_connector_joint_${id}" type="fixed">
+            <parent link="${parent}" />
+            <child link="${suffix}_leg_connector_${id}" />
             <origin rpy="0 0 0" xyz="0 0 0" />
-        </visual>
-        </link>
-        <joint name="${suffix}_y_hip_${id}" type="revolute">
-            <axis xyz="0 0 -1" />
-            <limit effort="1000" lower="-.1" upper="0.6" velocity="0.5" />
-            <parent link="${parent}"/>
-            <child link="${suffix}_y_hip_${id}"/>
-            <origin rpy="0 0 0" xyz="0 ${reflect * waist_length/2} 0" />
-        </joint>
-        <link name="${suffix}_p_hip_${id}">
-        </link>
-        <joint name="${suffix}_p_hip_${id}" type="revolute">
-            <axis xyz="${reflect} 0 0" />
-            <limit effort="1000" lower="-0.4" upper="3.3" velocity="0.5" />
-            <parent link="${suffix}_y_hip_${id}"/>
-            <child link="${suffix}_p_hip_${id}"/>
+        </joint>
+        <link name="${suffix}_leg_${id}">
+            <visual>
+                <geometry>
+                    <cylinder length="${leg_length}" radius="${limb_radius}" />
+                </geometry>
+                <material name="yellow-skin" />
+                <origin rpy="0 0 0" xyz="0 0 -${leg_length / 2}" />
+            </visual>
+            <collision>
+                <geometry>
+                    <cylinder length="${leg_length}" radius="${limb_radius}" />
+                </geometry>
+                <origin rpy="0 0 0" xyz="0 0 -${leg_length / 2}" />
+            </collision>
+            <visual>
+                <geometry>
+                    <sphere radius="${limb_radius}" />
+                </geometry>
+                <material name="yellow-skin-dark" />
+                <origin rpy="0 0 0" xyz="0 0 -${leg_length}" />
+            </visual>
+            <collision>
+                <geometry>
+                    <sphere radius="${limb_radius}" />
+                </geometry>
+                <origin rpy="0 0 0" xyz="0 0 -${leg_length}" />
+            </collision>
+        </link>
+        <joint name="${suffix}_leg_${id}" type="prismatic">
+            <parent link="${suffix}_leg_connector_${id}" />
+            <child link="${suffix}_leg_${id}" />
+            <axis xyz="0 0 1" />
+            <limit effort="1000.0" lower="0" upper="0.5" velocity="0.5" />
             <origin rpy="0 0 0" xyz="0 0 0" />
         </joint>
-        <xacro:limb_segment name="${suffix}_hip_${id}"
-                     length = "${tight_length}"
-                     reflect="${reflect}"
-                     parent="${suffix}_p_hip_${id}"
-                     attachment_origin="0 0 0"
-                     attachment_rotation="0 0 0"
-                     joint_name="${suffix}_r_hip_${id}"
-                     joint_axis="0 -1 0"
-                     joint_min_limit="-.4"
-                     joint_max_limit="0.7" />
-        <xacro:limb_segment name="${suffix}_knee_${id}"
-                     length = "${tibia_length}"
-                     reflect="${reflect}"
-                     parent="${suffix}_hip_${id}"
-                     attachment_origin="0 0 -${tight_length}"
-                     attachment_rotation="0 0 0"
-                     joint_name="${suffix}_knee_${id}"
-                     joint_axis="0 -1 0"
-                     joint_min_limit="-2.5"
-                     joint_max_limit="0" />
-        <link name="${suffix}_ankle_${id}">
-        </link>
-        <joint name="${suffix}_ankle_${id}" type="fixed">
-            <parent link="${suffix}_knee_${id}"/>
-            <child link="${suffix}_ankle_${id}"/>
-            <origin rpy="0 0 0" xyz="0 0 -${tibia_length}" />
-        </joint>
     </xacro:macro>
-    <xacro:leg suffix="l" reflect="1" parent="body_${id}" />
-    <xacro:leg suffix="r" reflect="-1" parent="body_${id}" />
+    <xacro:single_leg suffix="l" parent="body_${id}" />
 </robot>

Commit message: Updated human with no legs urdf.

File: urdf/human-no-legs.xacro (robot description, xacro)
@@ -30,12 +30,48 @@
         <color rgba="0 0 0 1" />
     </material>
-    <!--***********-->
-    <!-- <link name="world" /> -->
-    <link name="body_${id}">
-    </link>
-    <!-- <joint name="base_joint" type="fixed">
+    <!-- Ground link -->
+    <link name="world" />
+    <link name="fixed_leg_${id}">
+        <visual>
+            <geometry>
+                <cylinder length="${leg_length}" radius="${limb_radius}" />
+            </geometry>
+            <material name="yellow-skin" />
+            <origin rpy="0 0 0" xyz="0 0 ${leg_length / 2}" />
+        </visual>
+        <collision>
+            <geometry>
+                <cylinder length="${leg_length}" radius="${limb_radius}" />
+            </geometry>
+            <origin rpy="0 0 0" xyz="0 0 ${leg_length / 2}" />
+        </collision>
+    </link>
+    <joint name="fixed_leg_joint_${id}" type="fixed">
         <parent link="world" />
-        <child link="body_${id}" />
-    </joint> -->
+        <child link="fixed_leg_${id}" />
+        <origin rpy="0 0 0" xyz="0 0 0" />
+    </joint>
+    <link name="leg_${id}">
+        <visual>
+            <geometry>
+                <sphere radius="${limb_radius}"/>
+            </geometry>
+            <material name="yellow-skin" />
+            <origin rpy="0 0 0" xyz="0 0 0" />
+        </visual>
+        <collision>
+            <geometry>
+                <sphere radius="${limb_radius}"/>
+            </geometry>
+            <origin rpy="0 0 0" xyz="0 0 0" />
+        </collision>
+    </link>
+    <joint name="leg_crouch_joint_${id}" type="prismatic">
+        <parent link="fixed_leg_${id}" />
+        <child link="leg_${id}" />
+        <axis xyz="0 0 1" />
+        <limit effort="1000.0" lower="-0.5" upper="0.0" velocity="0.5" />
+        <origin rpy="0 0 0" xyz="0 0 ${leg_length}" />
+    </joint>
     <link name="waist_${id}">
     </link>
@@ -88,12 +124,12 @@
         <origin rpy="0 0 0" xyz="0 0 ${torso_height}" />
     </joint>
-    <joint name="waist_${id}_z" type="revolute">
+    <joint name="waist_rot_${id}" type="revolute">
         <axis xyz="0 0 1" />
         <limit effort="1000" lower="-.4" upper="0.4" velocity="0.5" />
-        <parent link="body_${id}"/>
+        <parent link="leg_${id}"/>
         <child link="waist_intermediate_${id}"/>
         <origin rpy="0 0 0" xyz="0 0 0" />
     </joint>
-    <joint name="waist_${id}" type="revolute">
+    <joint name="waist_bend_${id}" type="revolute">
         <axis xyz="0 1 0" />
         <limit effort="1000" lower="-.2" upper="1." velocity="0.5" />
@@ -263,61 +299,3 @@
     <xacro:arm suffix="l" reflect="1" parent="torso_${id}" />
     <xacro:arm suffix="r" reflect="-1" parent="torso_${id}" />
-    <xacro:macro name="single_leg" params="suffix parent">
-        <link name="${suffix}_leg_connector_${id}">
-            <visual>
-                <geometry>
-                    <sphere radius="${limb_radius}" />
-                </geometry>
-                <material name="yellow-skin-dark" />
-                <origin rpy="0 0 0" xyz="0 0 0" />
-            </visual>
-            <collision>
-                <geometry>
-                    <sphere radius="${limb_radius}" />
-                </geometry>
-                <origin rpy="0 0 0" xyz="0 0 0" />
-            </collision>
-        </link>
-        <joint name="${suffix}_leg_connector_joint_${id}" type="fixed">
-            <parent link="${parent}" />
-            <child link="${suffix}_leg_connector_${id}" />
-            <origin rpy="0 0 0" xyz="0 0 0" />
-        </joint>
-        <link name="${suffix}_leg_${id}">
-            <visual>
-                <geometry>
-                    <cylinder length="${leg_length}" radius="${limb_radius}" />
-                </geometry>
-                <material name="yellow-skin" />
-                <origin rpy="0 0 0" xyz="0 0 -${leg_length / 2}" />
-            </visual>
-            <collision>
-                <geometry>
-                    <cylinder length="${leg_length}" radius="${limb_radius}" />
-                </geometry>
-                <origin rpy="0 0 0" xyz="0 0 -${leg_length / 2}" />
-            </collision>
-            <visual>
-                <geometry>
-                    <sphere radius="${limb_radius}" />
-                </geometry>
-                <material name="yellow-skin-dark" />
-                <origin rpy="0 0 0" xyz="0 0 -${leg_length}" />
-            </visual>
-            <collision>
-                <geometry>
-                    <sphere radius="${limb_radius}" />
-                </geometry>
-                <origin rpy="0 0 0" xyz="0 0 -${leg_length}" />
-            </collision>
-        </link>
-        <joint name="${suffix}_leg_${id}" type="prismatic">
-            <parent link="${suffix}_leg_connector_${id}" />
-            <child link="${suffix}_leg_${id}" />
-            <axis xyz="0 0 1" />
-            <limit effort="1000.0" lower="0" upper="0.5" velocity="0.5" />
-            <origin rpy="0 0 0" xyz="0 0 0" />
-        </joint>
-    </xacro:macro>
-    <xacro:single_leg suffix="l" parent="body_${id}" />
 </robot>

Commit message: Updating URDF

File: urdf/human-no-legs.xacro (robot description, xacro)
@@ -20,4 +20,5 @@
     <xacro:property name="leg_length" value="${size_unit*2 + size_unit*1.5}" />
     <xacro:property name="limb_radius" value="0.03" />
+    <xacro:property name="hand_size" value="${limb_radius*2}" />
     <!-- Materials -->
     <material name="yellow-skin">
@@ -296,4 +297,35 @@
             <origin rpy="0 0 0" xyz="0 0 -${forearm_length}" />
         </joint>
+        <link name="${suffix}_wrist_intermediate_r_${id}">
+        </link>
+        <joint name="${suffix}_wrist_r_${id}" type="revolute">
+            <axis xyz="0 1 0" />
+            <limit effort="1000" lower="-0.4" upper="0.4" velocity="0.5" />
+            <parent link="${suffix}_wrist_${id}" />
+            <child link="${suffix}_wrist_intermediate_r_${id}" />
+            <origin rpy="0 ${pi / 2} 0" xyz="0 0 0" />
+        </joint>
+        <link name="${suffix}_wrist_intermediate_y_${id}">
+            <visual>
+                <geometry>
+                    <box size="${hand_size} ${hand_size} ${hand_size}" />
+                </geometry>
+                <material name="yellow-skin-dark" />
+                <origin rpy="0 0 0" xyz="0 0 0" />
+            </visual>
+            <collision>
+                <geometry>
+                    <box size="${hand_size} ${hand_size} ${hand_size}" />
+                </geometry>
+                <origin rpy="0 0 0" xyz="0 0 0" />
+            </collision>
+        </link>
+        <joint name="${suffix}_wrist_y_${id}" type="revolute">
+            <axis xyz="0 0 1" />
+            <limit effort="1000" lower="-0.2" upper="0.2" velocity="0.5" />
+            <parent link="${suffix}_wrist_intermediate_r_${id}" />
+            <child link="${suffix}_wrist_intermediate_y_${id}" />
+            <origin rpy="0 0 0" xyz="0 0 0" />
+        </joint>
     </xacro:macro>
     <xacro:arm suffix="l" reflect="1" parent="torso_${id}" />

Commit message: Updating urdf.

File: urdf/human-no-legs.xacro (robot description, xacro)
@@ -13,5 +13,5 @@
     <xacro:property name="neck_shoulder_length" value="${size_unit*0.8}" />
     <xacro:property name="upperarm_length" value="${size_unit*1.6}" />
-    <xacro:property name="forearm_length" value="${size_unit}" />
+    <xacro:property name="forearm_length" value="${size_unit*1.3}" />
     <xacro:property name="torso_height" value="${size_unit*2.75}" />
     <xacro:property name="waist_length" value="${size_unit*1.2}" />
@@ -19,5 +19,5 @@
     <xacro:property name="tibia_length" value="${size_unit*2}" />
     <xacro:property name="leg_length" value="${size_unit*2 + size_unit*1.5}" />
-    <xacro:property name="limb_radius" value="0.03" />f
+    <xacro:property name="limb_radius" value="0.03" />
     <xacro:property name="hand_size" value="${limb_radius*2}" />
     <!-- Materials -->

Commit message: Updating human description.

File: urdf/human-no-legs.xacro (robot description, xacro)
@@ -330,8 +330,10 @@
             </collision>
         </link>
-        <joint name="${suffix}_wrist_intermediate_fixed_${id}" type="fixed">
+        <joint name="${suffix}_wrist_intermediate_fixed_${id}" type="prismatic">
             <parent link="${suffix}_wrist_intermediate_y_${id}" />
             <child link="${suffix}_wrist_intermediate_fixed_${id}" />
-            <origin rpy="0 0 0" xyz="0 0 0" />
+            <axis xyz="1 0 0" />
+            <origin rpy="0 0 0" xyz="0 0 0" />
+            <limit effort="1000.0" lower="0.0" upper="0.001" velocity="0.5" />
         </joint>
     </xacro:macro>
